Commit message: Add files via upload

File: test_node/urdf/camera.urdf.xacro (robot description, xacro)
@@ -5,4 +5,8 @@
                 <sphere radius="0.001" />
             </geometry>
+            <origin xyz="0.0 0.0 0.0" rpy="0.0 0.0 0.0" />
+            <material name="yellow">
+                <color rgba="0.5 0.3 0.0 1" />
+            </material>
         </visual>
         <collision>
@@ -14,5 +18,5 @@
         <inertial>
             <origin xyz="0 0 0" />
-            <mass value="0" />
+            <mass value="6" />
             <inertia ixx="1" ixy="0" ixz="0" iyy="1" iyz="0" izz="1" />
         </inertial>
@@ -23,4 +27,8 @@
                 <box size="0.01 0.15 0.1" />
             </geometry>
+            <origin xyz="0.0 0.0 0.0" rpy="0.0 0.0 0.0" />
+            <material name = "yellow">
+                <color rgba="0.5 0.3 0.0 1" />
+            </material>
         </visual>
         <collision>
@@ -39,5 +47,5 @@
         <parent link="base_link"/>
         <child link="camera_box" />
-        <origin xyz="0 0 1" rpy="0 0 0" />
+        <origin xyz="0 0 1" rpy="0 0.7854 0" />
         <axis xyz="0 0 0" />
     </joint>

File: test_node/urdf/mycar.urdf (robot description, URDF)
Before this commit: robot mycar, 3 links, 2 joints
Links:
- removed link base_footprint
- removed link camera
- link base_link: mass None -> 6; geometry collision box size=0.5 0.2 0.1; visual box size=0.5 0.2 0.1
Joints:
- removed joint base_link2base_footprint
- removed joint camera2baselink
